Commit message: better gestures

File: llm_robot_bridge/urdf/robot.urdf (robot description, URDF)
Before this commit: robot service_robot, 22 links, 21 joints
Links:
- removed link back_caster_link
- removed link front_caster_link
- removed link left_hand_link
- removed link left_shoulder_pitch_link
- removed link left_shoulder_roll_link
- removed link left_wheel_link
- removed link left_wrist_pitch_link
- removed link right_hand_link
- removed link right_shoulder_pitch_link
- removed link right_shoulder_roll_link
- removed link right_wheel_link
- removed link right_wrist_pitch_link
- added link front_caster, mass 0.5; collision sphere radius=0.05; visual sphere radius=0.05
- added link left_elbow_link, mass 0.5; visual sphere radius=0.04
- added link left_index_p1, mass 0.02; visual cylinder length=0.04 radius=0.008
- added link left_index_p2, mass 0.015; visual cylinder length=0.03 radius=0.007
- added link left_index_p3, mass 0.01; visual cylinder length=0.02 radius=0.006
- added link left_middle_p1, mass 0.02; visual cylinder length=0.042 radius=0.008400000000000001
- added link left_middle_p2, mass 0.015; visual cylinder length=0.0315 radius=0.007350000000000001
- added link left_middle_p3, mass 0.01; visual cylinder length=0.021 radius=0.0063
- added link left_palm_link, mass 0.5; visual box size=0.05 0.1 0.02
- added link left_pinky_p1, mass 0.02; visual cylinder length=0.032 radius=0.0064
- added link left_pinky_p2, mass 0.015; visual cylinder length=0.024 radius=0.005600000000000001
- added link left_pinky_p3, mass 0.01; visual cylinder length=0.016 radius=0.0048000000000000004
- added link left_ring_p1, mass 0.02; visual cylinder length=0.04 radius=0.008
- added link left_ring_p2, mass 0.015; visual cylinder length=0.03 radius=0.007
- added link left_ring_p3, mass 0.01; visual cylinder length=0.02 radius=0.006
- added link left_sh_pitch_link, mass 1.0; visual sphere radius=0.05
- added link left_sh_roll_link, mass 1.0; visual sphere radius=0.05
- added link left_thumb_p1, mass 0.03; visual cylinder length=0.05500000000000001 radius=0.011000000000000001
- added link left_thumb_p2, mass 0.02; visual cylinder length=0.033 radius=0.0099
- added link left_wheel, mass 2.0; collision cylinder length=0.05 radius=0.1; visual cylinder length=0.05 radius=0.1
- added link rear_caster, mass 0.5; collision sphere radius=0.05; visual sphere radius=0.05
- added link right_elbow_link, mass 0.5; visual sphere radius=0.04
- added link right_index_p1, mass 0.02; visual cylinder length=0.04 radius=0.008
- added link right_index_p2, mass 0.015; visual cylinder length=0.03 radius=0.007
- added link right_index_p3, mass 0.01; visual cylinder length=0.02 radius=0.006
- added link right_middle_p1, mass 0.02; visual cylinder length=0.042 radius=0.008400000000000001
- added link right_middle_p2, mass 0.015; visual cylinder length=0.0315 radius=0.007350000000000001
- added link right_middle_p3, mass 0.01; visual cylinder length=0.021 radius=0.0063
- added link right_palm_link, mass 0.5; visual box size=0.05 0.1 0.02
- added link right_pinky_p1, mass 0.02; visual cylinder length=0.032 radius=0.0064
- added link right_pinky_p2, mass 0.015; visual cylinder length=0.024 radius=0.005600000000000001
- added link right_pinky_p3, mass 0.01; visual cylinder length=0.016 radius=0.0048000000000000004
- added link right_ring_p1, mass 0.02; visual cylinder length=0.04 radius=0.008
- added link right_ring_p2, mass 0.015; visual cylinder length=0.03 radius=0.007
- added link right_ring_p3, mass 0.01; visual cylinder length=0.02 radius=0.006
- added link right_sh_pitch_link, mass 1.0; visual sphere radius=0.05
- added link right_sh_roll_link, mass 1.0; visual sphere radius=0.05
- added link right_thumb_p1, mass 0.03; visual cylinder length=0.05500000000000001 radius=0.011000000000000001
- added link right_thumb_p2, mass 0.02; visual cylinder length=0.033 radius=0.0099
- added link right_wheel, mass 2.0; collision cylinder length=0.05 radius=0.1; visual cylinder length=0.05 radius=0.1
- link base_link: geometry visual cylinder length=0.15 radius=0.3
- link head_link: mass 1.0 -> 1.5; geometry visual box size=0.05 0.3 0.2; visual cylinder length=0.01 radius=0.025
- link left_forearm_link: mass 0.1 -> 1.5; geometry visual cylinder length=0.25 radius=0.035
- link left_upper_arm_link: mass 0.2 -> 2.0; geometry visual cylinder length=0.3 radius=0.04
- link left_wrist_roll_link: mass 0.02 -> 0.3; geometry visual sphere radius=0.035
- link right_forearm_link: mass 0.1 -> 1.5; geometry visual cylinder length=0.25 radius=0.035
- link right_upper_arm_link: mass 0.2 -> 2.0; geometry visual cylinder length=0.3 radius=0.04
- link right_wrist_roll_link: mass 0.02 -> 0.3; geometry visual sphere radius=0.035
- link torso_link: mass 12.0 -> 8.0; geometry visual cylinder length=0.5 radius=0.04; visual cylinder length=0.85 radius=0.08
Joints:
- removed joint back_caster_joint
- removed joint base_footprint_joint
- removed joint left_elbow_joint
- removed joint left_shoulder_pitch_joint
- removed joint left_shoulder_roll_joint
- removed joint left_shoulder_yaw_joint
- removed joint left_wrist_pitch_joint
- removed joint left_wrist_roll_joint
- removed joint left_wrist_yaw_joint
- removed joint right_elbow_joint
- removed joint right_shoulder_pitch_joint
- removed joint right_shoulder_roll_joint
- removed joint right_shoulder_yaw_joint
- removed joint right_wrist_pitch_joint
- removed joint right_wrist_roll_joint
- removed joint right_wrist_yaw_joint
- removed joint torso_joint
- added joint base_joint: type fixed, parent base_footprint, child base_link, origin xyz=0 0 0.05 rpy=0 0 0
- added joint left_elbow: type revolute, parent left_upper_arm_link, child left_elbow_link, origin xyz=0 0 -0.3 rpy=0 0 0, axis 0 1 0, limit lower=-2.5 upper=0.0 effort=40 velocity=2.0
- added joint left_index_j1: type revolute, parent left_palm_link, child left_index_p1, origin xyz=0.05 -0.035 0 rpy=0 0 0, axis 0 1 0, limit lower=0 upper=1.57 effort=2 velocity=3
- added joint left_index_j2: type revolute, parent left_index_p1, child left_index_p2, origin xyz=0.04 0 0 rpy=0 0 0, axis 0 1 0, limit lower=0 upper=1.57 effort=2 velocity=3
- added joint left_index_j3: type revolute, parent left_index_p2, child left_index_p3, origin xyz=0.03 0 0 rpy=0 0 0, axis 0 1 0, limit lower=0 upper=1.57 effort=2 velocity=3
- added joint left_middle_j1: type revolute, parent left_palm_link, child left_middle_p1, origin xyz=0.05 -0.01 0 rpy=0 0 0, axis 0 1 0, limit lower=0 upper=1.57 effort=2 velocity=3
- added joint left_middle_j2: type revolute, parent left_middle_p1, child left_middle_p2, origin xyz=0.042 0 0 rpy=0 0 0, axis 0 1 0, limit lower=0 upper=1.57 effort=2 velocity=3
- added joint left_middle_j3: type revolute, parent left_middle_p2, child left_middle_p3, origin xyz=0.0315 0 0 rpy=0 0 0, axis 0 1 0, limit lower=0 upper=1.57 effort=2 velocity=3
- added joint left_pinky_j1: type revolute, parent left_palm_link, child left_pinky_p1, origin xyz=0.05 0.04 0 rpy=0 0 0, axis 0 1 0, limit lower=0 upper=1.57 effort=2 velocity=3
- added joint left_pinky_j2: type revolute, parent left_pinky_p1, child left_pinky_p2, origin xyz=0.032 0 0 rpy=0 0 0, axis 0 1 0, limit lower=0 upper=1.57 effort=2 velocity=3
- added joint left_pinky_j3: type revolute, parent left_pinky_p2, child left_pinky_p3, origin xyz=0.024 0 0 rpy=0 0 0, axis 0 1 0, limit lower=0 upper=1.57 effort=2 velocity=3
- added joint left_ring_j1: type revolute, parent left_palm_link, child left_ring_p1, origin xyz=0.05 0.015 0 rpy=0 0 0, axis 0 1 0, limit lower=0 upper=1.57 effort=2 velocity=3
- added joint left_ring_j2: type revolute, parent left_ring_p1, child left_ring_p2, origin xyz=0.04 0 0 rpy=0 0 0, axis 0 1 0, limit lower=0 upper=1.57 effort=2 velocity=3
- added joint left_ring_j3: type revolute, parent left_ring_p2, child left_ring_p3, origin xyz=0.03 0 0 rpy=0 0 0, axis 0 1 0, limit lower=0 upper=1.57 effort=2 velocity=3
- added joint left_shoulder_pitch: type revolute, parent torso_link, child left_sh_pitch_link, origin xyz=0.0 0.25 0.75 rpy=0 0 0, axis 0 1 0, limit lower=-2.0 upper=2.0 effort=60 velocity=1.5
- added joint left_shoulder_roll: type revolute, parent left_sh_pitch_link, child left_sh_roll_link, origin xyz=0 0 0 rpy=0 0 0, axis 1 0 0, limit lower=-2.0 upper=2.0 effort=60 velocity=1.5
- added joint left_shoulder_yaw: type revolute, parent left_sh_roll_link, child left_upper_arm_link, origin xyz=0 0 0 rpy=0 0 0, axis 0 0 1, limit lower=-2.0 upper=2.0 effort=40 velocity=2.0
- added joint left_thumb_j1: type revolute, parent left_palm_link, child left_thumb_p1, origin xyz=0.025 -0.05 0 rpy=0 0 -0.785, axis 0 1 0, limit lower=0 upper=1.57 effort=3 velocity=3
- added joint left_thumb_j2: type revolute, parent left_thumb_p1, child left_thumb_p2, origin xyz=0.05500000000000001 0 0 rpy=0 0 0, axis 0 1 0, limit lower=0 upper=1.57 effort=3 velocity=3
- added joint left_wrist_pitch: type revolute, parent left_elbow_link, child left_forearm_link, origin xyz=0 0 0 rpy=0 0 0, axis 0 1 0, limit lower=-1.57 upper=1.57 effort=20 velocity=2.5
- added joint left_wrist_roll: type revolute, parent left_forearm_link, child left_wrist_roll_link, origin xyz=0 0 -0.25 rpy=0 0 0, axis 1 0 0, limit lower=-1.57 upper=1.57 effort=20 velocity=2.5
- added joint left_wrist_yaw: type revolute, parent left_wrist_roll_link, child left_palm_link, origin xyz=0 0 -0.035 rpy=0 1.5708 0, axis 0 0 1, limit lower=-1.57 upper=1.57 effort=10 velocity=3.0
- added joint rear_caster_joint: type continuous, parent base_link, child rear_caster, origin xyz=-0.25 0 0.0 rpy=0 0 0, axis 1 1 1
- added joint right_elbow: type revolute, parent right_upper_arm_link, child right_elbow_link, origin xyz=0 0 -0.3 rpy=0 0 0, axis 0 1 0, limit lower=-2.5 upper=0.0 effort=40 velocity=2.0
- added joint right_index_j1: type revolute, parent right_palm_link, child right_index_p1, origin xyz=0.05 0.035 0 rpy=0 0 0, axis 0 1 0, limit lower=0 upper=1.57 effort=2 velocity=3
- added joint right_index_j2: type revolute, parent right_index_p1, child right_index_p2, origin xyz=0.04 0 0 rpy=0 0 0, axis 0 1 0, limit lower=0 upper=1.57 effort=2 velocity=3
- added joint right_index_j3: type revolute, parent right_index_p2, child right_index_p3, origin xyz=0.03 0 0 rpy=0 0 0, axis 0 1 0, limit lower=0 upper=1.57 effort=2 velocity=3
- added joint right_middle_j1: type revolute, parent right_palm_link, child right_middle_p1, origin xyz=0.05 0.01 0 rpy=0 0 0, axis 0 1 0, limit lower=0 upper=1.57 effort=2 velocity=3
- added joint right_middle_j2: type revolute, parent right_middle_p1, child right_middle_p2, origin xyz=0.042 0 0 rpy=0 0 0, axis 0 1 0, limit lower=0 upper=1.57 effort=2 velocity=3
- added joint right_middle_j3: type revolute, parent right_middle_p2, child right_middle_p3, origin xyz=0.0315 0 0 rpy=0 0 0, axis 0 1 0, limit lower=0 upper=1.57 effort=2 velocity=3
- added joint right_pinky_j1: type revolute, parent right_palm_link, child right_pinky_p1, origin xyz=0.05 -0.04 0 rpy=0 0 0, axis 0 1 0, limit lower=0 upper=1.57 effort=2 velocity=3
- added joint right_pinky_j2: type revolute, parent right_pinky_p1, child right_pinky_p2, origin xyz=0.032 0 0 rpy=0 0 0, axis 0 1 0, limit lower=0 upper=1.57 effort=2 velocity=3
- added joint right_pinky_j3: type revolute, parent right_pinky_p2, child right_pinky_p3, origin xyz=0.024 0 0 rpy=0 0 0, axis 0 1 0, limit lower=0 upper=1.57 effort=2 velocity=3
- added joint right_ring_j1: type revolute, parent right_palm_link, child right_ring_p1, origin xyz=0.05 -0.015 0 rpy=0 0 0, axis 0 1 0, limit lower=0 upper=1.57 effort=2 velocity=3
- added joint right_ring_j2: type revolute, parent right_ring_p1, child right_ring_p2, origin xyz=0.04 0 0 rpy=0 0 0, axis 0 1 0, limit lower=0 upper=1.57 effort=2 velocity=3
- added joint right_ring_j3: type revolute, parent right_ring_p2, child right_ring_p3, origin xyz=0.03 0 0 rpy=0 0 0, axis 0 1 0, limit lower=0 upper=1.57 effort=2 velocity=3
- added joint right_shoulder_pitch: type revolute, parent torso_link, child right_sh_pitch_link, origin xyz=0.0 -0.25 0.75 rpy=0 0 0, axis 0 1 0, limit lower=-2.0 upper=2.0 effort=60 velocity=1.5
- added joint right_shoulder_roll: type revolute, parent right_sh_pitch_link, child right_sh_roll_link, origin xyz=0 0 0 rpy=0 0 0, axis 1 0 0, limit lower=-2.0 upper=2.0 effort=60 velocity=1.5
- added joint right_shoulder_yaw: type revolute, parent right_sh_roll_link, child right_upper_arm_link, origin xyz=0 0 0 rpy=0 0 0, axis 0 0 1, limit lower=-2.0 upper=2.0 effort=40 velocity=2.0
- added joint right_thumb_j1: type revolute, parent right_palm_link, child right_thumb_p1, origin xyz=0.025 0.05 0 rpy=0 0 0.785, axis 0 1 0, limit lower=0 upper=1.57 effort=3 velocity=3
- added joint right_thumb_j2: type revolute, parent right_thumb_p1, child right_thumb_p2, origin xyz=0.05500000000000001 0 0 rpy=0 0 0, axis 0 1 0, limit lower=0 upper=1.57 effort=3 velocity=3
- added joint right_wrist_pitch: type revolute, parent right_elbow_link, child right_forearm_link, origin xyz=0 0 0 rpy=0 0 0, axis 0 1 0, limit lower=-1.57 upper=1.57 effort=20 velocity=2.5
- added joint right_wrist_roll: type revolute, parent right_forearm_link, child right_wrist_roll_link, origin xyz=0 0 -0.25 rpy=0 0 0, axis 1 0 0, limit lower=-1.57 upper=1.57 effort=20 velocity=2.5
- added joint right_wrist_yaw: type revolute, parent right_wrist_roll_link, child right_palm_link, origin xyz=0 0 -0.035 rpy=0 1.5708 0, axis 0 0 1, limit lower=-1.57 upper=1.57 effort=10 velocity=3.0
- added joint torso_lift_joint: type prismatic, parent base_link, child torso_link, origin xyz=0 0 0.15 rpy=0 0 0, axis 0 0 1, limit lower=0.0 upper=0.3 effort=1000 velocity=0.5
- joint front_caster_joint: axis (none) -> 1 1 1; child front_caster_link -> front_caster; origin xyz=0.18 0 -0.10 rpy=0 0 0 -> xyz=0.25 0 0.0 rpy=0 0 0; type fixed -> continuous
- joint head_joint: origin xyz=0 0 0.475 rpy=0 0 0 -> xyz=0 0 0.95 rpy=0 0 0
- joint left_wheel_joint: axis 0 0 1 -> 0 1 0; child left_wheel_link -> left_wheel; origin xyz=0 0.26 -0.05 rpy=-1.5708 0 0 -> xyz=0 0.35 0.05 rpy=0 0 0
- joint right_wheel_joint: axis 0 0 1 -> 0 1 0; child right_wheel_link -> right_wheel; origin xyz=0 -0.26 -0.05 rpy=-1.5708 0 0 -> xyz=0 -0.35 0.05 rpy=0 0 0
