Commit message: better gestures

File: llm_robot_bridge/urdf/robot.urdf.xacro (robot description, xacro)
@@ -1,385 +1,323 @@
 <?xml version="1.0"?>
-<robot name="service_robot" xmlns:xacro="http://www.ros.org/wiki/xacro">
-  <material name="dark_grey"><color rgba="0.2 0.2 0.2 1.0"/></material>
-  <material name="white"><color rgba="0.9 0.9 0.9 1.0"/></material>
-  <material name="blue"><color rgba="0.0 0.4 0.8 1.0"/></material>
-  <material name="orange"><color rgba="1.0 0.5 0.0 1.0"/></material>
-  <material name="black"><color rgba="0.0 0.0 0.0 1.0"/></material>
-  <link name="base_footprint"/>
-  <joint name="base_footprint_joint" type="fixed">
-    <parent link="base_footprint"/>
-    <child link="base_link"/>
-    <origin xyz="0 0 0.15" rpy="0 0 0"/>
-  </joint>
-  <link name="base_link">
-    <inertial>
-      <mass value="15.0"/>
-      <origin xyz="0 0 0" rpy="0 0 0"/>
-      <inertia ixx="0.2625" ixy="0" ixz="0" iyy="0.2625" iyz="0" izz="0.46875"/>
-    </inertial>
-    <visual>
-      <geometry><cylinder radius="0.25" length="0.15"/></geometry>
-      <material name="dark_grey"/>
-    </visual>
-    <collision>
-      <geometry><cylinder radius="0.25" length="0.15"/></geometry>
-    </collision>
-  </link>
-  <joint name="left_wheel_joint" type="continuous">
-    <parent link="base_link"/>
-    <child link="left_wheel_link"/>
-    <origin xyz="0 0.26 -0.05" rpy="-1.5708 0 0"/>
-    <axis xyz="0 0 1"/>
-  </joint>
-  <link name="left_wheel_link">
-    <inertial>
-      <mass value="1.5"/>
-      <inertia ixx="0.0041" ixy="0" ixz="0" iyy="0.0041" iyz="0" izz="0.0075"/>
-    </inertial>
-    <visual>
-      <geometry><cylinder radius="0.10" length="0.05"/></geometry>
-      <material name="black"/>
-    </visual>
-    <collision>
-      <geometry><cylinder radius="0.10" length="0.05"/></geometry>
-    </collision>
-  </link>
-  <joint name="right_wheel_joint" type="continuous">
-    <parent link="base_link"/>
-    <child link="right_wheel_link"/>
-    <origin xyz="0 -0.26 -0.05" rpy="-1.5708 0 0"/>
-    <axis xyz="0 0 1"/>
-  </joint>
-  <link name="right_wheel_link">
-    <inertial>
-      <mass value="1.5"/>
-      <inertia ixx="0.0041" ixy="0" ixz="0" iyy="0.0041" iyz="0" izz="0.0075"/>
-    </inertial>
-    <visual>
-      <geometry><cylinder radius="0.10" length="0.05"/></geometry>
-      <material name="black"/>
-    </visual>
-    <collision>
-      <geometry><cylinder radius="0.10" length="0.05"/></geometry>
-    </collision>
-  </link>
-  <joint name="front_caster_joint" type="fixed">
-    <parent link="base_link"/>
-    <child link="front_caster_link"/>
-    <origin xyz="0.18 0 -0.10" rpy="0 0 0"/>
-  </joint>
-  <link name="front_caster_link">
-    <inertial>
-      <mass value="0.5"/>
-      <inertia ixx="0.0002" ixy="0" ixz="0" iyy="0.0002" iyz="0" izz="0.0002"/>
-    </inertial>
-    <visual>
-      <geometry><sphere radius="0.05"/></geometry>
-      <material name="dark_grey"/>
-    </visual>
-    <collision>
-      <geometry><sphere radius="0.05"/></geometry>
-    </collision>
-  </link>
-  <joint name="back_caster_joint" type="fixed">
-    <parent link="base_link"/>
-    <child link="back_caster_link"/>
-    <origin xyz="-0.18 0 -0.10" rpy="0 0 0"/>
-  </joint>
-  <link name="back_caster_link">
-    <inertial>
-      <mass value="0.5"/>
-      <inertia ixx="0.0002" ixy="0" ixz="0" iyy="0.0002" iyz="0" izz="0.0002"/>
-    </inertial>
-    <visual>
-      <geometry><sphere radius="0.05"/></geometry>
-      <material name="dark_grey"/>
-    </visual>
-    <collision>
-      <geometry><sphere radius="0.05"/></geometry>
-    </collision>
-  </link>
-  <joint name="torso_joint" type="fixed">
-    <parent link="base_link"/>
-    <child link="torso_link"/>
-    <origin xyz="0 0 0.475" rpy="0 0 0"/>
-  </joint>
-  <link name="torso_link">
-    <inertial>
-      <mass value="12.0"/>
-      <origin xyz="0 0 0" rpy="0 0 0"/>
-      <inertia ixx="0.68" ixy="0" ixz="0" iyy="0.73" iyz="0" izz="0.13"/>
-    </inertial>
-    <visual>
-      <geometry><box size="0.3 0.2 0.8"/></geometry>
-      <material name="white"/>
-    </visual>
-    <collision>
-      <geometry><box size="0.3 0.2 0.8"/></geometry>
-    </collision>
-  </link>
-  <joint name="head_joint" type="fixed">
-    <parent link="torso_link"/>
-    <child link="head_link"/>
-    <origin xyz="0 0 0.475" rpy="0 0 0"/>
-  </joint>
-  <link name="head_link">
-    <inertial>
-      <mass value="1.0"/>
-      <inertia ixx="0.002" ixy="0" ixz="0" iyy="0.002" iyz="0" izz="0.002"/>
-    </inertial>
-    <visual>
-      <geometry><box size="0.15 0.15 0.15"/></geometry>
-      <material name="blue"/>
-    </visual>
-    <collision>
-      <geometry><box size="0.15 0.15 0.15"/></geometry>
-    </collision>
-  </link>
-  <xacro:macro name="arm_7dof" params="side reflect">
-    <joint name="${side}_shoulder_pitch_joint" type="revolute">
-      <parent link="torso_link"/>
-      <child link="${side}_shoulder_pitch_link"/>
-      <origin xyz="0 ${reflect * 0.16} 0.3" rpy="0 0 0"/>
-      <axis xyz="0 1 0"/>
-      <limit lower="-3.14159" upper="3.14159" effort="40.0" velocity="2.0"/>
-      <dynamics damping="0.1" friction="0.1"/>
+<robot xmlns:xacro="http://www.ros.org/wiki/xacro" name="dual_arm_service_bot">
+    <material name="white_mat">
+        <color rgba="1.0 1.0 1.0 1.0"/>
+    </material>
+    <material name="dark_grey">
+        <color rgba="0.2 0.2 0.2 1.0"/>
+    </material>
+    <material name="black_mat">
+        <color rgba="0.0 0.0 0.0 1.0"/>
+    </material>
+    <material name="blue_mat">
+        <color rgba="0.0 0.4 0.8 1.0"/>
+    </material>
+    <xacro:macro name="box_inertia" params="m w h d">
+        <inertial>
+            <mass value="${m}"/>
+            <inertia ixx="${(m/12)*(h*h + d*d)}" ixy="0" ixz="0" iyy="${(m/12)*(w*w + d*d)}" iyz="0" izz="${(m/12)*(w*w + h*h)}"/>
+        </inertial>
+    </xacro:macro>
+    <xacro:macro name="cyl_inertia" params="m r h">
+        <inertial>
+            <mass value="${m}"/>
+            <inertia ixx="${(m/12)*(3*r*r + h*h)}" ixy="0" ixz="0" iyy="${(m/12)*(3*r*r + h*h)}" iyz="0" izz="${0.5*m*r*r}"/>
+        </inertial>
+    </xacro:macro>
+    <xacro:macro name="sph_inertia" params="m r">
+        <inertial>
+            <mass value="${m}"/>
+            <inertia ixx="${0.4*m*r*r}" ixy="0" ixz="0" iyy="${0.4*m*r*r}" iyz="0" izz="${0.4*m*r*r}"/>
+        </inertial>
+    </xacro:macro>
+    <xacro:macro name="pos_ctrl" params="joint">
+        <gazebo>
+            <plugin filename="gz-sim-joint-position-controller-system" name="gz::sim::systems::JointPositionController">
+                <joint_name>${joint}</joint_name>
+                <p_gain>20.0</p_gain>
+                <i_gain>0.1</i_gain>
+                <d_gain>1.0</d_gain>
+            </plugin>
+        </gazebo>
+    </xacro:macro>
+    <xacro:macro name="finger" params="prefix name xyz rpy scale:=1.0">
+        <link name="${prefix}_${name}_p1">
+            <visual><origin xyz="${0.02 * scale} 0 0" rpy="0 1.5708 0"/><geometry><cylinder radius="${0.008 * scale}" length="${0.04 * scale}"/></geometry><material name="black_mat"/></visual>
+            <xacro:cyl_inertia m="0.02" r="${0.008 * scale}" h="${0.04 * scale}"/>
+        </link>
+        <gazebo reference="${prefix}_${name}_p1"><material>Gazebo/Black</material></gazebo>
+        <joint name="${prefix}_${name}_j1" type="revolute">
+            <parent link="${prefix}_palm_link"/>
+            <child link="${prefix}_${name}_p1"/>
+            <origin xyz="${xyz}" rpy="${rpy}"/>
+            <axis xyz="0 1 0"/>
+            <limit lower="0" upper="1.57" effort="2" velocity="3"/>
+        </joint>
+        <xacro:pos_ctrl joint="${prefix}_${name}_j1"/>
+        <link name="${prefix}_${name}_p2">
+            <visual><origin xyz="${0.015 * scale} 0 0" rpy="0 1.5708 0"/><geometry><cylinder radius="${0.007 * scale}" length="${0.03 * scale}"/></geometry><material name="black_mat"/></visual>
+            <xacro:cyl_inertia m="0.015" r="${0.007 * scale}" h="${0.03 * scale}"/>
+        </link>
+        <gazebo reference="${prefix}_${name}_p2"><material>Gazebo/Black</material></gazebo>
+        <joint name="${prefix}_${name}_j2" type="revolute">
+            <parent link="${prefix}_${name}_p1"/>
+            <child link="${prefix}_${name}_p2"/>
+            <origin xyz="${0.04 * scale} 0 0" rpy="0 0 0"/>
+            <axis xyz="0 1 0"/>
+            <limit lower="0" upper="1.57" effort="2" velocity="3"/>
+        </joint>
+        <xacro:pos_ctrl joint="${prefix}_${name}_j2"/>
+        <link name="${prefix}_${name}_p3">
+            <visual><origin xyz="${0.01 * scale} 0 0" rpy="0 1.5708 0"/><geometry><cylinder radius="${0.006 * scale}" length="${0.02 * scale}"/></geometry><material name="black_mat"/></visual>
+            <xacro:cyl_inertia m="0.01" r="${0.006 * scale}" h="${0.02 * scale}"/>
+        </link>
+        <gazebo reference="${prefix}_${name}_p3"><material>Gazebo/Black</material></gazebo>
+        <joint name="${prefix}_${name}_j3" type="revolute">
+            <parent link="${prefix}_${name}_p2"/>
+            <child link="${prefix}_${name}_p3"/>
+            <origin xyz="${0.03 * scale} 0 0" rpy="0 0 0"/>
+            <axis xyz="0 1 0"/>
+            <limit lower="0" upper="1.57" effort="2" velocity="3"/>
+        </joint>
+        <xacro:pos_ctrl joint="${prefix}_${name}_j3"/>
+    </xacro:macro>
+    <xacro:macro name="thumb" params="prefix xyz rpy scale:=1.0">
+        <link name="${prefix}_thumb_p1">
+            <visual><origin xyz="${0.025 * scale} 0 0" rpy="0 1.5708 0"/><geometry><cylinder radius="${0.01 * scale}" length="${0.05 * scale}"/></geometry><material name="black_mat"/></visual>
+            <xacro:cyl_inertia m="0.03" r="${0.01 * scale}" h="${0.05 * scale}"/>
+        </link>
+        <gazebo reference="${prefix}_thumb_p1"><material>Gazebo/Black</material></gazebo>
+        <joint name="${prefix}_thumb_j1" type="revolute">
+            <parent link="${prefix}_palm_link"/>
+            <child link="${prefix}_thumb_p1"/>
+            <origin xyz="${xyz}" rpy="${rpy}"/>
+            <axis xyz="0 1 0"/>
+            <limit lower="0" upper="1.57" effort="3" velocity="3"/>
+        </joint>
+        <xacro:pos_ctrl joint="${prefix}_thumb_j1"/>
+        <link name="${prefix}_thumb_p2">
+            <visual><origin xyz="${0.015 * scale} 0 0" rpy="0 1.5708 0"/><geometry><cylinder radius="${0.009 * scale}" length="${0.03 * scale}"/></geometry><material name="black_mat"/></visual>
+            <xacro:cyl_inertia m="0.02" r="${0.009 * scale}" h="${0.03 * scale}"/>
+        </link>
+        <gazebo reference="${prefix}_thumb_p2"><material>Gazebo/Black</material></gazebo>
+        <joint name="${prefix}_thumb_j2" type="revolute">
+            <parent link="${prefix}_thumb_p1"/>
+            <child link="${prefix}_thumb_p2"/>
+            <origin xyz="${0.05 * scale} 0 0" rpy="0 0 0"/>
+            <axis xyz="0 1 0"/>
+            <limit lower="0" upper="1.57" effort="3" velocity="3"/>
+        </joint>
+        <xacro:pos_ctrl joint="${prefix}_thumb_j2"/>
+    </xacro:macro>
+    <xacro:macro name="arm" params="prefix reflect">
+        <link name="${prefix}_sh_pitch_link"><visual><geometry><sphere radius="0.05"/></geometry><material name="white_mat"/></visual><xacro:sph_inertia m="1.0" r="0.05"/></link>
+        <gazebo reference="${prefix}_sh_pitch_link"><material>Gazebo/White</material></gazebo>
+        <joint name="${prefix}_shoulder_pitch" type="revolute">
+            <parent link="torso_link"/>
+            <child link="${prefix}_sh_pitch_link"/>
+            <origin xyz="0.0 ${reflect * 0.25} 0.75" rpy="0 0 0"/> <axis xyz="0 1 0"/>
+            <limit lower="-2.0" upper="2.0" effort="60" velocity="1.5"/>
+        </joint>
+        <xacro:pos_ctrl joint="${prefix}_shoulder_pitch"/>
+        <link name="${prefix}_sh_roll_link"><visual><geometry><sphere radius="0.05"/></geometry><material name="white_mat"/></visual><xacro:sph_inertia m="1.0" r="0.05"/></link>
+        <gazebo reference="${prefix}_sh_roll_link"><material>Gazebo/White</material></gazebo>
+        <joint name="${prefix}_shoulder_roll" type="revolute">
+            <parent link="${prefix}_sh_pitch_link"/>
+            <child link="${prefix}_sh_roll_link"/>
+            <origin xyz="0 0 0" rpy="0 0 0"/>
+            <axis xyz="1 0 0"/>
+            <limit lower="-2.0" upper="2.0" effort="60" velocity="1.5"/>
+        </joint>
+        <xacro:pos_ctrl joint="${prefix}_shoulder_roll"/>
+        <link name="${prefix}_upper_arm_link">
+            <visual><origin xyz="0 0 -0.15" rpy="0 0 0"/><geometry><cylinder radius="0.04" length="0.3"/></geometry><material name="white_mat"/></visual>
+            <xacro:cyl_inertia m="2.0" r="0.04" h="0.3"/>
+        </link>
+        <gazebo reference="${prefix}_upper_arm_link"><material>Gazebo/White</material></gazebo>
+        <joint name="${prefix}_shoulder_yaw" type="revolute">
+            <parent link="${prefix}_sh_roll_link"/>
+            <child link="${prefix}_upper_arm_link"/>
+            <origin xyz="0 0 0" rpy="0 0 0"/>
+            <axis xyz="0 0 1"/>
+            <limit lower="-2.0" upper="2.0" effort="40" velocity="2.0"/>
+        </joint>
+        <gazebo>
+            <plugin filename="gz-sim-joint-position-controller-system" name="gz::sim::systems::JointPositionController">
+                <joint_name>${prefix}_shoulder_yaw</joint_name>
+                <p_gain>20.0</p_gain>
+                <i_gain>0.1</i_gain>
+                <d_gain>1.0</d_gain>
+                <initial_position>${reflect * 1.57}</initial_position>
+            </plugin>
+        </gazebo>
+        <link name="${prefix}_elbow_link"><visual><geometry><sphere radius="0.04"/></geometry><material name="white_mat"/></visual><xacro:sph_inertia m="0.5" r="0.04"/></link>
+        <gazebo reference="${prefix}_elbow_link"><material>Gazebo/White</material></gazebo>
+        <!-- elbow bend (existing) -->
+        <joint name="${prefix}_elbow" type="revolute">
+            <parent link="${prefix}_upper_arm_link"/>
+            <child link="${prefix}_elbow_link"/>
+            <origin xyz="0 0 -0.3" rpy="0 0 0"/>
+            <axis xyz="0 1 0"/>
+            <limit lower="-2.5" upper="0.0" effort="40" velocity="2.0"/>
+        </joint>
+        <xacro:pos_ctrl joint="${prefix}_elbow"/>
+        <!-- elbow roll — new intermediate link so forearm can swing up/down -->
+        <link name="${prefix}_elbow_roll_link">
+            <visual><geometry><sphere radius="0.035"/></geometry><material name="white_mat"/></visual>
+            <xacro:sph_inertia m="0.3" r="0.035"/>
+        </link>
+        <gazebo reference="${prefix}_elbow_roll_link"><material>Gazebo/White</material></gazebo>
+        <joint name="${prefix}_elbow_roll" type="revolute">
+            <parent link="${prefix}_elbow_link"/>
+            <child link="${prefix}_elbow_roll_link"/>
+            <origin xyz="0 0 0" rpy="0 0 0"/>
+            <axis xyz="1 0 0"/>
+            <limit lower="-1.57" upper="1.57" effort="40" velocity="2.0"/>
+        </joint>
+        <xacro:pos_ctrl joint="${prefix}_elbow_roll"/>
+        <link name="${prefix}_forearm_link">
+            <visual><origin xyz="0 0 -0.125" rpy="0 0 0"/><geometry><cylinder radius="0.035" length="0.25"/></geometry><material name="white_mat"/></visual>
+            <xacro:cyl_inertia m="1.5" r="0.035" h="0.25"/>
+        </link>
+        <gazebo reference="${prefix}_forearm_link"><material>Gazebo/White</material></gazebo>
+        <joint name="${prefix}_wrist_pitch" type="revolute">
+            <parent link="${prefix}_elbow_roll_link"/>
+            <child link="${prefix}_forearm_link"/>
+            <origin xyz="0 0 0" rpy="0 0 0"/>
+            <axis xyz="0 1 0"/>
+            <limit lower="-1.57" upper="1.57" effort="20" velocity="2.5"/>
+        </joint>
+        <xacro:pos_ctrl joint="${prefix}_wrist_pitch"/>
+        <link name="${prefix}_wrist_roll_link"><visual><geometry><sphere radius="0.035"/></geometry><material name="white_mat"/></visual><xacro:sph_inertia m="0.3" r="0.035"/></link>
+        <gazebo reference="${prefix}_wrist_roll_link"><material>Gazebo/White</material></gazebo>
+        <joint name="${prefix}_wrist_roll" type="revolute">
+            <parent link="${prefix}_forearm_link"/>
+            <child link="${prefix}_wrist_roll_link"/>
+            <origin xyz="0 0 -0.25" rpy="0 0 0"/>
+            <axis xyz="1 0 0"/>
+            <limit lower="-1.57" upper="1.57" effort="20" velocity="2.5"/>
+        </joint>
+        <xacro:pos_ctrl joint="${prefix}_wrist_roll"/>
+        <link name="${prefix}_palm_link">
+            <visual><origin xyz="0.025 0 0" rpy="0 0 0"/><geometry><box size="0.05 0.1 0.02"/></geometry><material name="black_mat"/></visual>
+            <xacro:box_inertia m="0.5" w="0.05" h="0.1" d="0.02"/>
+        </link>
+        <gazebo reference="${prefix}_palm_link"><material>Gazebo/Black</material></gazebo>
+        <joint name="${prefix}_wrist_yaw" type="revolute">
+            <parent link="${prefix}_wrist_roll_link"/>
+            <child link="${prefix}_palm_link"/>
+            <origin xyz="0 0 -0.035" rpy="0 1.5708 0"/>
+            <axis xyz="0 0 1"/>
+            <limit lower="-1.57" upper="1.57" effort="10" velocity="3.0"/>
+        </joint>
+        <xacro:pos_ctrl joint="${prefix}_wrist_yaw"/>
+        <xacro:finger prefix="${prefix}" name="index"  xyz="0.05 ${reflect * -0.035} 0" rpy="0 0 0" scale="1.0"/>
+        <xacro:finger prefix="${prefix}" name="middle" xyz="0.05 ${reflect * -0.010} 0" rpy="0 0 0" scale="1.05"/>
+        <xacro:finger prefix="${prefix}" name="ring"   xyz="0.05 ${reflect * 0.015} 0" rpy="0 0 0" scale="1.0"/>
+        <xacro:finger prefix="${prefix}" name="pinky"  xyz="0.05 ${reflect * 0.040} 0" rpy="0 0 0" scale="0.8"/>
+        <xacro:thumb prefix="${prefix}" xyz="0.025 ${reflect * -0.05} 0" rpy="0 0 ${reflect * -0.785}" scale="1.1"/>
+    </xacro:macro>
+    <link name="base_footprint"/>
+    <link name="base_link">
+        <visual><origin xyz="0 0 0.075" rpy="0 0 0"/><geometry><cylinder radius="0.3" length="0.15"/></geometry><material name="white_mat"/></visual>
+        <xacro:cyl_inertia m="15.0" r="0.3" h="0.15"/>
+    </link>
+    <gazebo reference="base_link"><material>Gazebo/White</material></gazebo>
+    <joint name="base_joint" type="fixed">
+        <parent link="base_footprint"/>
+        <child link="base_link"/>
+        <origin xyz="0 0 0.05" rpy="0 0 0"/>
     </joint>
-    <link name="${side}_shoulder_pitch_link">
-      <inertial>
-        <mass value="0.05"/>
-        <inertia ixx="0.0001" ixy="0" ixz="0" iyy="0.0001" iyz="0" izz="0.0001"/>
-      </inertial>
-      <visual>
-        <geometry><sphere radius="0.01"/></geometry>
-        <material name="orange"/>
-      </visual>
+    <xacro:macro name="wheel" params="prefix y_dir">
+        <link name="${prefix}_wheel">
+            <visual><origin xyz="0 0 0" rpy="1.5708 0 0"/><geometry><cylinder radius="0.1" length="0.05"/></geometry><material name="dark_grey"/></visual>
+            <collision><origin xyz="0 0 0" rpy="1.5708 0 0"/><geometry><cylinder radius="0.1" length="0.05"/></geometry></collision>
+            <xacro:cyl_inertia m="2.0" r="0.1" h="0.05"/>
+        </link>
+        <gazebo reference="${prefix}_wheel"><material>Gazebo/DarkGrey</material></gazebo>
+        <joint name="${prefix}_wheel_joint" type="continuous">
+            <parent link="base_link"/>
+            <child link="${prefix}_wheel"/>
+            <origin xyz="0 ${y_dir * 0.35} 0.05" rpy="0 0 0"/>
+            <axis xyz="0 1 0"/>
+            <dynamics damping="0.1" friction="0.1"/>
+        </joint>
+    </xacro:macro>
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