Commit message: feat: Added more gestures

File: llm_robot_bridge/urdf/robot.urdf (robot description, URDF)
Before this commit: robot dual_arm_service_bot, 50 links, 49 joints
Links:
- added link left_elbow_roll_link, mass 0.3; visual sphere radius=0.035
- added link right_elbow_roll_link, mass 0.3; visual sphere radius=0.035
- link head_link: geometry visual box size=0.01 0.08 0.03; visual box size=0.05 0.3 0.2
- link torso_link: geometry visual cylinder length=0.25 radius=0.06; visual cylinder length=0.3 radius=0.12
Joints:
- added joint left_elbow_roll: type revolute, parent left_elbow_link, child left_elbow_roll_link, origin xyz=0 0 0 rpy=0 0 0, axis 1 0 0, limit lower=-1.57 upper=1.57 effort=40 velocity=2.0
- added joint right_elbow_roll: type revolute, parent right_elbow_link, child right_elbow_roll_link, origin xyz=0 0 0 rpy=0 0 0, axis 1 0 0, limit lower=-1.57 upper=1.57 effort=40 velocity=2.0
- joint base_joint: origin xyz=0 0 0.05 rpy=0 0 0 -> xyz=0 0 0.1 rpy=0 0 0
- joint front_caster_joint: axis 1 1 1 -> (none); origin xyz=0.25 0 0.0 rpy=0 0 0 -> xyz=0.25 0 -0.05 rpy=0 0 0; type continuous -> fixed
- joint left_wheel_joint: origin xyz=0 0.35 0.05 rpy=0 0 0 -> xyz=0 0.35 0.0 rpy=0 0 0
- joint left_wrist_pitch: parent left_elbow_link -> left_elbow_roll_link
- joint rear_caster_joint: axis 1 1 1 -> (none); origin xyz=-0.25 0 0.0 rpy=0 0 0 -> xyz=-0.25 0 -0.05 rpy=0 0 0; type continuous -> fixed
- joint right_wheel_joint: origin xyz=0 -0.35 0.05 rpy=0 0 0 -> xyz=0 -0.35 0.0 rpy=0 0 0
- joint right_wrist_pitch: parent right_elbow_link -> right_elbow_roll_link

File: llm_robot_bridge/urdf/robot.urdf.xacro (robot description, xacro)
@@ -227,5 +227,5 @@
         <parent link="base_footprint"/>
         <child link="base_link"/>
-        <origin xyz="0 0 0.05" rpy="0 0 0"/>
+        <origin xyz="0 0 0.1" rpy="0 0 0"/>
     </joint>
     <xacro:macro name="wheel" params="prefix y_dir">
@@ -235,9 +235,16 @@
             <xacro:cyl_inertia m="2.0" r="0.1" h="0.05"/>
         </link>
-        <gazebo reference="${prefix}_wheel"><material>Gazebo/DarkGrey</material></gazebo>
+        <!-- 💡 UPDATED GAZEBO REFERENCE BLOCK WITH SURFACE FRICTION OVERRIDES -->
+        <gazebo reference="${prefix}_wheel">
+            <material>Gazebo/DarkGrey</material>
+            <mu1>1.5</mu1>
+            <mu2>1.5</mu2>
+            <kp>1000000.0</kp>
+            <kd>1.0</kd>
+        </gazebo>
         <joint name="${prefix}_wheel_joint" type="continuous">
             <parent link="base_link"/>
             <child link="${prefix}_wheel"/>
-            <origin xyz="0 ${y_dir * 0.35} 0.05" rpy="0 0 0"/>
+            <origin xyz="0 ${y_dir * 0.35} 0.0" rpy="0 0 0"/>
             <axis xyz="0 1 0"/>
             <dynamics damping="0.1" friction="0.1"/>
@@ -256,5 +263,5 @@
             <parent link="base_link"/>
             <child link="${prefix}_caster"/>
-            <origin xyz="${x_dir * 0.25} 0 0.0" rpy="0 0 0"/>
+            <origin xyz="${x_dir * 0.25} 0 -0.05" rpy="0 0 0"/>
         </joint>
     </xacro:macro>
@@ -313,10 +320,10 @@
             <wheel_radius>0.1</wheel_radius>
             <odom_publish_frequency>50</odom_publish_frequency>
-            <max_linear_acceleration>1</max_linear_acceleration>
-            <max_angular_acceleration>2</max_angular_acceleration>
-            <topic>/cmd_vel</topic>
-            <odom_topic>/model/dual_arm_service_bot/odometry</odom_topic>
+            <max_linear_acceleration>2.0</max_linear_acceleration>
+            <max_angular_acceleration>4.0</max_angular_acceleration>
+            <topic>/model/dual_arm_service_bot/cmd_vel</topic>
+            <robot_base_frame>base_footprint</robot_base_frame>
+            <odom_topic>/model/dual_arm_service_bot/odom</odom_topic>
             <tf_topic>/model/dual_arm_service_bot/tf</tf_topic>
-            <robot_base_frame>base_footprint</robot_base_frame>
         </plugin>
     </gazebo>
